Commit message: Working driver implementation

File: webots_driver/urdf/panda.urdf (robot description, URDF)
Before this commit: robot panda, 12 links, 11 joints
Joints:
- joint panda_finger_joint2: mimic joint=panda_finger_joint1 -> (none)

File: webots_driver/urdf/panda_hand.ros2_control.xacro (robot description, xacro)
@@ -12,6 +12,5 @@
             </joint>
             <joint name="panda_finger_joint2">
-                <param name="mimic">panda_finger_joint1</param>
-                <param name="multiplier">1</param>
+                <param name="initial_position">0.0</param>
                 <command_interface name="position" />
                 <state_interface name="position"/>
